File: docs/schematics/Nemesis-Mod.sch (KiCad schematic (older format))
At the start: 10 parts

Commit message: Adding Adafruit I2C FRAM breakout packages.
Parts:
- added FRAM1: Adafruit_I2C_FRAM_Breakout, symbol Nemesis-Mod:Adafruit_I2C_FRAM_Breakout
- MCU: symbol Nemesis-Mod:Adafruit_Feather_M0 -> Nemesis-Mod-rescue:Adafruit_Feather_M0-Nemesis-Mod
Connections:
- wire segments 102 -> 116

Commit message: Initial adding software reset button support.
Parts:
- added AUTH_RESET: SW_Button, symbol Switch:SW_Push
Connections:
- wire segments 116 -> 121
Changed lines of the file:
@@
 Wire Wire Line
 	4750 5250 4450 5250
+$Comp
+L Switch:SW_Push AUTH_RESET
+U 1 1 5D15A0F1
+P 1900 3150
+F 0 "AUTH_RESET" H 1900 3435 50  0000 C CNN
+F 1 "SW_Button" H 1900 3344 50  0000 C CNN
+F 2 "" H 1900 3350 50  0001 C CNN
+F 3 "~" H 1900 3350 50  0001 C CNN
+	1    1900 3150
+	1    0    0    -1
+$EndComp
+Wire Wire Line
+	3050 4200 2350 4200
+Wire Wire Line
+	2950 3150 2100 3150
+Connection ~ 2950 3150
+Wire Wire Line
+	2350 4200 2350 3250
+Wire Wire Line
+	2350 3250 1700 3250
+Wire Wire Line
+	1700 3250 1700 3150
 $EndSCHEMATC

Commit message: Updating schematic.
Parts:
- renumbered AUTH_RESET to RESET
Connections:
- wire segments 121 -> 118
Changed lines of the file:
@@
 	6900 4850 6900 5450
 Wire Wire Line
-	6750 5450 6750 5150
-Wire Wire Line
-	6750 5150 7050 5150
-Wire Wire Line
-	7050 5150 7050 4850
-Wire Wire Line
-	7050 5450 7050 5300
-Wire Wire Line
-	7050 5300 4650 5300
-Wire Wire Line
-	4650 5300 4650 3900
+	6750 5450 6750 5100
+Wire Wire Line
+	6750 5100 7050 5100
+Wire Wire Line
+	7050 5100 7050 4850
+Wire Wire Line
+	7050 5450 7050 5200
+Wire Wire Line
+	7050 5200 4650 5200
+Wire Wire Line
+	4650 5200 4650 3900
 Wire Wire Line
 	4650 3900 4450 3900
@@
 U 1 1 5CEA8643
 P 3100 6250
-F 0 "Rev_Trigger" H 3100 6535 50  0000 C CNN
-F 1 "SW_Push_SPDT" H 3100 6444 50  0000 C CNN
+F 0 "Rev_Trigger" H 3100 5900 50  0000 C CNN
+F 1 "SW_Push_SPDT" H 3100 6000 50  0000 C CNN
 F 2 "" H 3100 6250 50  0001 C CNN
 F 3 "~" H 3100 6250 50  0001 C CNN
@@
 L Switch:SW_Push_SPDT Firing_Trigger
 U 1 1 5CEA8EFA
-P 5050 6250
-F 0 "Firing_Trigger" H 5050 6535 50  0000 C CNN
-F 1 "SW_Push_SPDT" H 5050 6444 50  0000 C CNN
-F 2 "" H 5050 6250 50  0001 C CNN
-F 3 "~" H 5050 6250 50  0001 C CNN
-	1    5050 6250
+P 4800 6250
+F 0 "Firing_Trigger" H 4800 5900 50  0000 C CNN
+F 1 "SW_Push_SPDT" H 4800 6000 50  0000 C CNN
+F 2 "" H 4800 6250 50  0001 C CNN
+F 3 "~" H 4800 6250 50  0001 C CNN
+	1    4800 6250
 	1    0    0    -1
 $EndComp
@@
 	4550 4050 4550 5800
 Wire Wire Line
-	2750 6250 2900 6250
-Wire Wire Line
-	4550 5800 2750 5800
-Wire Wire Line
-	2750 5800 2750 6250
+	4550 5800 2900 5800
+Wire Wire Line
+	2900 5800 2900 6250
 Wire Wire Line
 	4600 4200 4600 6250
-Wire Wire Line
-	4600 6250 4850 6250
 Wire Wire Line
 	2850 3450 2850 4900
@@
 Connection ~ 2850 3450
 Wire Wire Line
-	5500 5750 5500 6150
-Wire Wire Line
-	5500 6150 5250 6150
+	5000 5750 5000 6150
 Wire Wire Line
 	2850 5750 3500 5750
 Connection ~ 3500 5750
 Wire Wire Line
-	3500 5750 5500 5750
+	3500 5750 5000 5750
 Wire Wire Line
 	3050 3150 2950 3150
@@
 	3600 6350 3300 6350
 Wire Wire Line
-	3600 5700 5600 5700
-Wire Wire Line
-	5600 5700 5600 6350
-Wire Wire Line
-	5600 6350 5250 6350
+	3600 5700 5100 5700
+Wire Wire Line
+	5100 5700 5100 6350
+Wire Wire Line
+	5100 6350 5000 6350
 Connection ~ 3600 5700
 Text Label 9300 3850 0    50   ~ 0
@@
 	4750 5250 4450 5250
 $Comp
-L Switch:SW_Push AUTH_RESET
+L Switch:SW_Push RESET
 U 1 1 5D15A0F1
 P 1900 3150
-F 0 "AUTH_RESET" H 1900 3435 50  0000 C CNN
+F 0 "RESET" H 1900 3435 50  0000 C CNN
 F 1 "SW_Button" H 1900 3344 50  0000 C CNN
 F 2 "" H 1900 3350 50  0001 C CNN

Commit message: Updating the schematic.
Connections:
- wire segments 118 -> 117
Changed lines of the file:
@@
 L Device:Battery BATT
 U 1 1 5CE683D1
-P 9650 3550
-F 0 "BATT" H 9500 3550 50  0000 R CNN
-F 1 "3S LiPo Battery" H 9500 3650 50  0000 R CNN
-F 2 "" V 9650 3610 50  0001 C CNN
-F 3 "~" V 9650 3610 50  0001 C CNN
-	1    9650 3550
+P 9800 3550
+F 0 "BATT" H 9700 3550 50  0000 R CNN
+F 1 "3S LiPo Battery" H 9700 3650 50  0000 R CNN
+F 2 "" V 9800 3610 50  0001 C CNN
+F 3 "~" V 9800 3610 50  0001 C CNN
+	1    9800 3550
 	-1   0    0    1
 $EndComp
@@
 Connection ~ 9350 3350
 Wire Wire Line
-	9350 3350 9650 3350
-Wire Wire Line
-	9150 3750 9150 1900
+	9350 3350 9800 3350
 Wire Wire Line
 	9150 1900 7800 1900
 Wire Wire Line
 	7800 1900 7800 1800
-Connection ~ 9150 3750
-Wire Wire Line
-	9150 3750 9650 3750
 Wire Wire Line
 	5950 1700 2550 1700
@@
 	2850 3450 2850 4900
 Wire Wire Line
-	3500 5750 3500 6150
-Wire Wire Line
-	3500 6150 3300 6150
+	3300 5750 3300 6150
 Connection ~ 2850 3450
 Wire Wire Line
 	5000 5750 5000 6150
 Wire Wire Line
-	2850 5750 3500 5750
-Connection ~ 3500 5750
-Wire Wire Line
-	3500 5750 5000 5750
+	2850 5750 3300 5750
+Connection ~ 3300 5750
+Wire Wire Line
+	3300 5750 5000 5750
 Wire Wire Line
 	3050 3150 2950 3150
@@
 	2950 3150 2950 5000
 Wire Wire Line
-	2950 5700 3600 5700
-Wire Wire Line
-	3600 5700 3600 6350
-Wire Wire Line
-	3600 6350 3300 6350
-Wire Wire Line
-	3600 5700 5100 5700
+	2950 5700 3400 5700
+Wire Wire Line
+	3400 5700 3400 6350
+Wire Wire Line
+	3400 6350 3300 6350
+Wire Wire Line
+	3400 5700 5100 5700
 Wire Wire Line
 	5100 5700 5100 6350
 Wire Wire Line
 	5100 6350 5000 6350
-Connection ~ 3600 5700
-Text Label 9300 3850 0    50   ~ 0
+Connection ~ 3400 5700
+Text Label 9450 3850 0    50   ~ 0
 12awg
 Text Label 7750 3750 0    50   ~ 0
@@
 Wire Wire Line
 	1700 3250 1700 3150
+Wire Wire Line
+	9150 3750 9150 1900
+Wire Wire Line
+	9150 3750 9800 3750
+Connection ~ 9150 3750
 $EndSCHEMATC

Commit message: Correcting reset button connections.
Parts:
- added Resistor: 10K, symbol Device:R_Small_US
- RESET: value SW_Button -> Tactile_SW_Button
Connections:
- wire segments 117 -> 120
Changed lines of the file:
@@
 	4750 2600 2850 2600
-Wire Wire Line
-	2850 2600 2850 3450
 Wire Wire Line
 	2850 3450 3050 3450
@@
 Wire Wire Line
 	3300 5750 5000 5750
-Wire Wire Line
-	3050 3150 2950 3150
 Wire Wire Line
 	2950 3150 2950 5000
@@
 Wire Wire Line
 	4750 5250 4450 5250
+Wire Wire Line
+	9150 3750 9150 1900
+Wire Wire Line
+	9150 3750 9800 3750
+Connection ~ 9150 3750
+Wire Wire Line
+	2850 2600 2850 3450
+Wire Wire Line
+	2050 2800 2050 2900
+$Comp
+L Device:R_Small_US Resistor
+U 1 1 5D19815F
+P 2050 3050
+F 0 "Resistor" H 2100 3100 50  0000 L CNN
+F 1 "10K" H 2118 3005 50  0000 L CNN
+F 2 "" H 2050 3050 50  0001 C CNN
+F 3 "~" H 2050 3050 50  0001 C CNN
+	1    2050 3050
+	1    0    0    -1
+$EndComp
 $Comp
 L Switch:SW_Push RESET
 U 1 1 5D15A0F1
-P 1900 3150
-F 0 "RESET" H 1900 3435 50  0000 C CNN
-F 1 "SW_Button" H 1900 3344 50  0000 C CNN
-F 2 "" H 1900 3350 50  0001 C CNN
-F 3 "~" H 1900 3350 50  0001 C CNN
-	1    1900 3150
-	1    0    0    -1
-$EndComp
-Wire Wire Line
-	3050 4200 2350 4200
-Wire Wire Line
-	2950 3150 2100 3150
+P 1850 2800
+F 0 "RESET" H 1850 3085 50  0000 C CNN
+F 1 "Tactile_SW_Button" H 1850 2994 50  0000 C CNN
+F 2 "" H 1850 3000 50  0001 C CNN
+F 3 "~" H 1850 3000 50  0001 C CNN
+	1    1850 2800
+	1    0    0    -1
+$EndComp
+Wire Wire Line
+	2050 3150 2950 3150
 Connection ~ 2950 3150
 Wire Wire Line
-	2350 4200 2350 3250
-Wire Wire Line
-	2350 3250 1700 3250
-Wire Wire Line
-	1700 3250 1700 3150
-Wire Wire Line
-	9150 3750 9150 1900
-Wire Wire Line
-	9150 3750 9800 3750
-Connection ~ 9150 3750
+	2850 3450 1650 3450
+Wire Wire Line
+	1650 3450 1650 2800
+Wire Wire Line
+	2050 2900 1900 2900
+Wire Wire Line
+	1900 2900 1900 4200
+Connection ~ 2050 2900
+Wire Wire Line
+	2050 2900 2050 2950
+Wire Wire Line
+	1900 4200 3050 4200
+Wire Wire Line
+	2950 3150 3050 3150
 $EndSCHEMATC

Commit message: Updating schematics for new hardware.
Parts:
- MCU: value Adafruit_Feather_M0 -> Bluefruit_nRF52_Feather
Changed lines of the file:
@@
 EESchema Schematic File Version 4
-LIBS:Nemesis-Mod-cache
 EELAYER 29 0
 EELAYER END
@@
 $EndDescr
 $Comp
-L Nemesis-Mod-rescue:Adafruit_Feather_M0-Nemesis-Mod MCU
-U 1 1 5CE64CEC
-P 3750 4150
-F 0 "MCU" H 3750 5565 50  0000 C CNN
-F 1 "Adafruit_Feather_M0" H 3750 5474 50  0000 C CNN
-F 2 "" H 4400 2850 50  0001 C CNN
-F 3 "" H 4400 2850 50  0001 C CNN
-	1    3750 4150
-	1    0    0    -1
-$EndComp
-$Comp
 L Device:Battery BATT
 U 1 1 5CE683D1
@@
 	4650 5200 4650 3900
 Wire Wire Line
-	4650 3900 4450 3900
-Wire Wire Line
 	6750 4850 6750 5050
 Wire Wire Line
@@
 	5100 3800 5100 2550
 Wire Wire Line
-	5100 2550 2750 2550
-Wire Wire Line
-	2750 2550 2750 3600
-Wire Wire Line
 	2750 3600 3050 3600
 Wire Wire Line
 	3050 3750 2650 3750
-Wire Wire Line
-	2650 3750 2650 2500
 Wire Wire Line
 	2650 2500 5000 2500
@@
 	7800 1900 7800 1800
 Wire Wire Line
-	5950 1700 2550 1700
-Wire Wire Line
-	2550 1700 2550 3900
-Wire Wire Line
 	2550 3900 3050 3900
 Wire Wire Line
@@
 	4850 1400 4850 4350
 Wire Wire Line
-	4850 4350 4450 4350
-Wire Wire Line
 	5950 1500 2450 1500
 Wire Wire Line
-	2450 1500 2450 4050
-Wire Wire Line
 	2450 4050 3050 4050
-Wire Wire Line
-	2850 2600 2850 1200
 Wire Wire Line
 	2850 1200 5950 1200
@@
 $EndComp
 Wire Wire Line
-	4450 4200 4600 4200
-Wire Wire Line
 	4450 4050 4550 4050
-Wire Wire Line
-	4550 4050 4550 5800
 Wire Wire Line
 	4550 5800 2900 5800
@@
 Wire Wire Line
 	3300 5750 5000 5750
-Wire Wire Line
-	2950 3150 2950 5000
 Wire Wire Line
 	2950 5700 3400 5700
@@
 Wire Wire Line
 	1800 5000 2950 5000
-Connection ~ 2950 5000
 Wire Wire Line
 	2950 5000 2950 5700
@@
 	9150 3750 9800 3750
 Connection ~ 9150 3750
-Wire Wire Line
-	2850 2600 2850 3450
 Wire Wire Line
 	2050 2800 2050 2900
@@
 $EndComp
 Wire Wire Line
-	2050 3150 2950 3150
-Connection ~ 2950 3150
-Wire Wire Line
 	2850 3450 1650 3450
 Wire Wire Line
@@
 Wire Wire Line
 	2950 3150 3050 3150
+Connection ~ 2950 3150
+Connection ~ 2950 5000
+Wire Wire Line
+	4850 4350 4450 4350
+Wire Wire Line
+	4450 4200 4600 4200
+Wire Wire Line
+	4650 3900 4450 3900
+Wire Wire Line
+	5100 2550 2750 2550
+Wire Wire Line
+	5950 1700 2550 1700
+Wire Wire Line
+	2850 2600 2850 1200
+Wire Wire Line
+	2050 3150 2950 3150
+Wire Wire Line
+	4550 4050 4550 5800
+Wire Wire Line
+	2850 2600 2850 3450
+Wire Wire Line
+	2950 3150 2950 5000
+Wire Wire Line
+	2450 1500 2450 4050
+Wire Wire Line
+	2550 1700 2550 3900
+Wire Wire Line
+	2650 3750 2650 2500
+Wire Wire Line
+	2750 2550 2750 3600
+$Comp
+L Nemesis-Mod-rescue:Adafruit_Feather_M0-Nemesis-Mod MCU
+U 1 1 5CE64CEC
+P 3750 4150
+F 0 "MCU" H 3750 5565 50  0000 C CNN
+F 1 "Bluefruit_nRF52_Feather" H 3750 5474 50  0000 C CNN
+F 2 "" H 4400 2850 50  0001 C CNN
+F 3 "" H 4400 2850 50  0001 C CNN
+	1    3750 4150
+	1    0    0    -1
+$EndComp
 $EndSCHEMATC

Commit message: Updating schematics.
Parts:
- removed MCU: Bluefruit_nRF52_Feather, symbol Nemesis-Mod-rescue:Adafruit_Feather_M0-Nemesis-Mod
- added MCU: Adafruit_nRF52_Feather, symbol Nemesis-Mod:Adafruit_nRF52_Feather
Changed lines of the file:
@@
 EESchema Schematic File Version 4
+LIBS:Nemesis-Mod-cache
 EELAYER 29 0
 EELAYER END
@@
 Title "Nemesis Mod"
 Date "2019-05-22"
-Rev "v1.0"
+Rev "v1.1"
 Comp "https://github.com/jeff-winn/Nemesis-Mod"
 Comment1 "For more information please visit the project website:"
@@
 	2750 2550 2750 3600
 $Comp
-L Nemesis-Mod-rescue:Adafruit_Feather_M0-Nemesis-Mod MCU
-U 1 1 5CE64CEC
+L Nemesis-Mod:Adafruit_nRF52_Feather MCU
+U 1 1 5DBD8417
 P 3750 4150
 F 0 "MCU" H 3750 5565 50  0000 C CNN
-F 1 "Bluefruit_nRF52_Feather" H 3750 5474 50  0000 C CNN
+F 1 "Adafruit_nRF52_Feather" H 3750 5474 50  0000 C CNN
 F 2 "" H 4400 2850 50  0001 C CNN
 F 3 "" H 4400 2850 50  0001 C CNN

Commit message: Adding hopper lock to schematic.
Parts:
- added Power_Lock: Nerf_Hopper_Lock, symbol Nemesis-Mod:Nerf_Hopper_Lock
Connections:
- wire segments 120 -> 127
- no-connect marks 0 -> 31
Changed lines of the file:
@@
 	7050 5100 7050 4850
-Wire Wire Line
-	7050 5450 7050 5200
-Wire Wire Line
-	7050 5200 4650 5200
-Wire Wire Line
-	4650 5200 4650 3900
-Wire Wire Line
-	6750 4850 6750 5050
-Wire Wire Line
-	6750 5050 4750 5050
-Wire Wire Line
-	4750 5050 4750 2600
-Wire Wire Line
-	4750 2600 2850 2600
 Wire Wire Line
 	2850 3450 3050 3450
@@
 Wire Wire Line
 	2850 1200 5950 1200
-Connection ~ 2850 2600
 $Comp
 L Switch:SW_Push_SPDT Rev_Trigger
@@
 	4450 4200 4600 4200
 Wire Wire Line
-	4650 3900 4450 3900
-Wire Wire Line
 	5100 2550 2750 2550
 Wire Wire Line
 	5950 1700 2550 1700
 Wire Wire Line
-	2850 2600 2850 1200
-Wire Wire Line
 	2050 3150 2950 3150
 Wire Wire Line
 	4550 4050 4550 5800
-Wire Wire Line
-	2850 2600 2850 3450
 Wire Wire Line
 	2950 3150 2950 5000
@@
 	1    0    0    -1
 $EndComp
+$Comp
+L Nemesis-Mod:Nerf_Hopper_Lock Power_Lock
+U 1 1 5DDF54E1
+P 8200 6650
+F 0 "Power_Lock" H 8150 7750 50  0000 C CNN
+F 1 "Nerf_Hopper_Lock" H 8150 7850 50  0000 C CNN
+F 2 "" H 8200 7750 50  0001 C CNN
+F 3 "" H 8200 7750 50  0001 C CNN
+	1    8200 6650
+	1    0    0    -1
+$EndComp
+Wire Wire Line
+	7050 5450 7600 5450
+Wire Wire Line
+	7600 6250 8150 6250
+Wire Wire Line
+	7600 5450 7600 6250
+Wire Wire Line
+	2850 1200 2850 2600
+Wire Wire Line
+	6750 4850 6750 5050
+Wire Wire Line
+	6750 5050 7750 5050
+Wire Wire Line
+	7750 5050 7750 5750
+Wire Wire Line
+	8550 5750 8550 5350
+Wire Wire Line
+	8550 5350 4900 5350
+Wire Wire Line
+	4900 5350 4900 2600
+Wire Wire Line
+	4900 2600 2850 2600
+Connection ~ 2850 2600
+Wire Wire Line
+	2850 2600 2850 3450
+Wire Wire Line
+	8550 5950 8600 5950
+Wire Wire Line
+	8600 5950 8600 5300
+Wire Wire Line
+	8600 5300 4950 5300
+Wire Wire Line
+	4950 5300 4950 3900
+Wire Wire Line
+	4950 3900 4450 3900
+NoConn ~ 7750 5950
+NoConn ~ 6600 5450
+NoConn ~ 5300 4250
+NoConn ~ 5300 3950
+NoConn ~ 5300 3500
+NoConn ~ 5300 3200
+NoConn ~ 5300 3050
+NoConn ~ 5300 2900
+NoConn ~ 5300 2750
+NoConn ~ 5300 2600
+NoConn ~ 4450 3750
+NoConn ~ 4450 3600
+NoConn ~ 3050 3300
+NoConn ~ 3050 3000
+NoConn ~ 3050 4350
+NoConn ~ 3050 4500
+NoConn ~ 3050 4650
+NoConn ~ 3050 4800
+NoConn ~ 3050 4950
+NoConn ~ 3050 5100
+NoConn ~ 3050 5250
+NoConn ~ 1800 4800
+NoConn ~ 1800 4500
+NoConn ~ 1800 4400
+NoConn ~ 1800 4300
+NoConn ~ 6450 4850
+NoConn ~ 6600 4850
+NoConn ~ 5950 1900
+NoConn ~ 5950 1800
+NoConn ~ 5950 1600
+NoConn ~ 5950 1300
 $EndSCHEMATC
