File: docs/kicad/nemesis/flywheels.kicad_sch (KiCad schematic)
At the start: 3 parts, among them M1-M2 Pololu_G2_HighPower_18v18

Commit message: Correcting title block.
Other:
- title: Nemesis Mod -> Nemesis
Changed lines of the file:
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@@
   (paper "A4")
   (title_block
-    (title "Nemesis Mod")
+    (title "Nemesis")
     (date "2021-12-08")
     (rev "v2.0")
