File: docs/kicad/nemesis/main.kicad_sch (KiCad schematic)
At the start: 7 parts, among them P1 Pololu_5V_Step_Down_Regulator, SW1 SW1

Commit message: Correcting title block.
Other:
- title: Nemesis Mod -> Nemesis
Changed lines of the file:
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@@
   (paper "A4")
   (title_block
-    (title "Nemesis Mod")
+    (title "Nemesis")
     (date "2021-12-08")
     (rev "v2.0")
