File: docs/kicad/nemesis/softlock.kicad_sch (KiCad schematic)
At the start: 1 part, among them SW2 Nerf Hopper Open Button

Commit message: Correcting title block.
Other:
- title: Nemesis Mod -> Nemesis
Changed lines of the file:
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@@
   (paper "A4")
   (title_block
-    (title "Nemesis Mod")
+    (title "Nemesis")
     (date "2021-12-08")
     (rev "v2.0")
